File: src/OSI 600D Superboard II Cherry Solder Mask.kicad_pcb (KiCad board)
At the start: 2 copper layers, 301.5 x 367.3 mm, 128 parts, among them J2 CONN_SDA-41815_12_RA_MOL, J3 CONN_SDA-41815_12_RA_MOL, SW1 SW_Cherry_MX_1.00u_PCB, SW2 SW_Cherry_MX_1.00u_PCB, U41 CHR ROM, U70 7803, U8 6502

Commit message: more footprints for capacitors
Parts:
- added C39: C_Rect_L10.0mm_W3.0mm_P7.50mm_FKS3_FKP3, Capacitor_THT:C_Rect_L10.0mm_W3.0mm_P7.50mm_FKS3_FKP3, F.Cu at (383.4, 135.8)
- added C40: C_Rect_L10.0mm_W3.0mm_P7.50mm_FKS3_FKP3, Capacitor_THT:C_Rect_L10.0mm_W3.0mm_P7.50mm_FKS3_FKP3, F.Cu at (366.9, 135.8)
- added C41: C_Rect_L10.0mm_W3.0mm_P7.50mm_FKS3_FKP3, Capacitor_THT:C_Rect_L10.0mm_W3.0mm_P7.50mm_FKS3_FKP3, F.Cu at (350.4, 135.8)
- added C42: C_Rect_L10.0mm_W3.0mm_P7.50mm_FKS3_FKP3, Capacitor_THT:C_Rect_L10.0mm_W3.0mm_P7.50mm_FKS3_FKP3, F.Cu at (333.9, 135.8)
- added C43: C_Rect_L10.0mm_W3.0mm_P7.50mm_FKS3_FKP3, Capacitor_THT:C_Rect_L10.0mm_W3.0mm_P7.50mm_FKS3_FKP3, F.Cu at (317.4, 135.8)
- added C44: C_Rect_L10.0mm_W3.0mm_P7.50mm_FKS3_FKP3, Capacitor_THT:C_Rect_L10.0mm_W3.0mm_P7.50mm_FKS3_FKP3, F.Cu at (300.9, 135.8)
- added C45: C_Rect_L10.0mm_W3.0mm_P7.50mm_FKS3_FKP3, Capacitor_THT:C_Rect_L10.0mm_W3.0mm_P7.50mm_FKS3_FKP3, F.Cu at (284.4, 135.8)
- added C46: C_Rect_L10.0mm_W3.0mm_P7.50mm_FKS3_FKP3, Capacitor_THT:C_Rect_L10.0mm_W3.0mm_P7.50mm_FKS3_FKP3, F.Cu at (268.0, 135.8)
- added C47: C_Rect_L10.0mm_W3.0mm_P7.50mm_FKS3_FKP3, Capacitor_THT:C_Rect_L10.0mm_W3.0mm_P7.50mm_FKS3_FKP3, F.Cu at (238.2, 124.2)
Routing:
- net (no net): track 62584.9 -> 62585.1 mm, vias 2143 -> 2125
Other:
- board text added: "Origional by Grant (Klyball) Enhanced by Jon (Bambelweeny57)"
- board text removed: "C39"
- board text removed: "C40"
- board text removed: "C41"
- board text removed: "C42"
- board text removed: "C43"
- board text removed: "C44"
- board text removed: "C45"
- board text removed: "C46"
- board text removed: "C47"
- board text removed: "Origional by Grant (Klyball) Added to by Jon (Bambelweeny57)"
- board text removed: "U48"

Commit message: more footprints and added disc capacitor and fuse 3d models
Parts:
- removed the ? at (267.8, 94.9)
- added C10: C_Rect_L10.0mm_W3.0mm_P7.50mm_FKS3_FKP3, OSI:C_Rect_L10.0mm_W3.0mm_P7.50mm_FKS3_FKP3, F.Cu at (222.4, 36.6)
- added C12: C_Rect_L10.0mm_W3.0mm_P7.50mm_FKS3_FKP3, OSI:C_Rect_L10.0mm_W3.0mm_P7.50mm_FKS3_FKP3, F.Cu at (225.0, 62.9)
- added C21: C_Rect_L10.0mm_W3.0mm_P7.50mm_FKS3_FKP3, OSI:C_Rect_L10.0mm_W3.0mm_P7.50mm_FKS3_FKP3, F.Cu at (399.5, 272.9)
- added C22: C_Rect_L10.0mm_W3.0mm_P7.50mm_FKS3_FKP3, OSI:C_Rect_L10.0mm_W3.0mm_P7.50mm_FKS3_FKP3, F.Cu at (355.3, 249.8)
- added C23: C_Rect_L10.0mm_W3.0mm_P7.50mm_FKS3_FKP3, OSI:C_Rect_L10.0mm_W3.0mm_P7.50mm_FKS3_FKP3, F.Cu at (332.4, 251.1)
- added C24: C_Rect_L10.0mm_W3.0mm_P7.50mm_FKS3_FKP3, OSI:C_Rect_L10.0mm_W3.0mm_P7.50mm_FKS3_FKP3, F.Cu at (309.6, 249.7)
- added C25: C_Rect_L10.0mm_W3.0mm_P7.50mm_FKS3_FKP3, OSI:C_Rect_L10.0mm_W3.0mm_P7.50mm_FKS3_FKP3, F.Cu at (274.1, 277.5)
- added C26: C_Rect_L10.0mm_W3.0mm_P7.50mm_FKS3_FKP3, OSI:C_Rect_L10.0mm_W3.0mm_P7.50mm_FKS3_FKP3, F.Cu at (244.9, 277.5)
- added C27: C_Rect_L10.0mm_W3.0mm_P7.50mm_FKS3_FKP3, OSI:C_Rect_L10.0mm_W3.0mm_P7.50mm_FKS3_FKP3, F.Cu at (222.2, 277.5)
- added C28: C_Rect_L10.0mm_W3.0mm_P7.50mm_FKS3_FKP3, OSI:C_Rect_L10.0mm_W3.0mm_P7.50mm_FKS3_FKP3, F.Cu at (199.4, 277.5)
- added C29: C_Rect_L10.0mm_W3.0mm_P7.50mm_FKS3_FKP3, OSI:C_Rect_L10.0mm_W3.0mm_P7.50mm_FKS3_FKP3, F.Cu at (176.5, 277.5)
- added C30: C_Rect_L10.0mm_W3.0mm_P7.50mm_FKS3_FKP3, OSI:C_Rect_L10.0mm_W3.0mm_P7.50mm_FKS3_FKP3, F.Cu at (153.7, 277.5)
- added C51: C_Rect_L10.0mm_W3.0mm_P7.50mm_FKS3_FKP3, OSI:C_Rect_L10.0mm_W3.0mm_P7.50mm_FKS3_FKP3, F.Cu at (200.2, 91.5)
- added C56: C_Rect_L10.0mm_W3.0mm_P7.50mm_FKS3_FKP3, OSI:C_Rect_L10.0mm_W3.0mm_P7.50mm_FKS3_FKP3, F.Cu at (333.1, 195.3)
- added C57: C_Disc_D10.0mm_W2.5mm_P5.00mm, Capacitor_THT:C_Disc_D10.0mm_W2.5mm_P5.00mm, F.Cu at (126.4, 109.0)
- added C6: C_Rect_L10.0mm_W3.0mm_P7.50mm_FKS3_FKP3, OSI:C_Rect_L10.0mm_W3.0mm_P7.50mm_FKS3_FKP3, F.Cu at (208.3, 74.3)
- added C60: C_Rect_L10.0mm_W3.0mm_P7.50mm_FKS3_FKP3, OSI:C_Rect_L10.0mm_W3.0mm_P7.50mm_FKS3_FKP3, F.Cu at (148.3, 320.7)
- added C61: C_Rect_L10.0mm_W3.0mm_P7.50mm_FKS3_FKP3, OSI:C_Rect_L10.0mm_W3.0mm_P7.50mm_FKS3_FKP3, F.Cu at (143.7, 320.7)
- added C62: C_Rect_L10.0mm_W3.0mm_P7.50mm_FKS3_FKP3, OSI:C_Rect_L10.0mm_W3.0mm_P7.50mm_FKS3_FKP3, F.Cu at (127.7, 382.9)
- added C65: C_Rect_L10.0mm_W3.0mm_P7.50mm_FKS3_FKP3, OSI:C_Rect_L10.0mm_W3.0mm_P7.50mm_FKS3_FKP3, F.Cu at (146.6, 137.9)
- added C68: C_Rect_L10.0mm_W3.0mm_P7.50mm_FKS3_FKP3, OSI:C_Rect_L10.0mm_W3.0mm_P7.50mm_FKS3_FKP3, F.Cu at (129.8, 306.8)
- added C8: C_Rect_L10.0mm_W3.0mm_P7.50mm_FKS3_FKP3, OSI:C_Rect_L10.0mm_W3.0mm_P7.50mm_FKS3_FKP3, F.Cu at (126.9, 101.8)
- added F1: 5A, OSI:Fuseholder_Clip-6.3x32mm_Littelfuse_102_Inline_P34.21x7.62mm_D2.54mm_Horizontal, F.Cu at (270.5, 66.8)
- added R1: R_Axial_DIN0207_L6.3mm_D2.5mm_P2.54mm_Vertical, Resistor_THT:R_Axial_DIN0207_L6.3mm_D2.5mm_P2.54mm_Vertical, F.Cu at (343.7, 277.5)
- added R10: R_Axial_DIN0207_L6.3mm_D2.5mm_P2.54mm_Vertical, Resistor_THT:R_Axial_DIN0207_L6.3mm_D2.5mm_P2.54mm_Vertical, F.Cu at (300.6, 277.5)
- added R11: R_Axial_DIN0207_L6.3mm_D2.5mm_P2.54mm_Vertical, Resistor_THT:R_Axial_DIN0207_L6.3mm_D2.5mm_P2.54mm_Vertical, F.Cu at (294.3, 277.5)
- added R2: R_Axial_DIN0207_L6.3mm_D2.5mm_P2.54mm_Vertical, Resistor_THT:R_Axial_DIN0207_L6.3mm_D2.5mm_P2.54mm_Vertical, F.Cu at (339.9, 277.5)
- added R3: R_Axial_DIN0207_L6.3mm_D2.5mm_P2.54mm_Vertical, Resistor_THT:R_Axial_DIN0207_L6.3mm_D2.5mm_P2.54mm_Vertical, F.Cu at (336.1, 277.5)
- added R4: R_Axial_DIN0207_L6.3mm_D2.5mm_P2.54mm_Vertical, Resistor_THT:R_Axial_DIN0207_L6.3mm_D2.5mm_P2.54mm_Vertical, F.Cu at (332.4, 277.5)
- added R5: R_Axial_DIN0207_L6.3mm_D2.5mm_P2.54mm_Vertical, Resistor_THT:R_Axial_DIN0207_L6.3mm_D2.5mm_P2.54mm_Vertical, F.Cu at (328.6, 277.5)
- added R6: R_Axial_DIN0207_L6.3mm_D2.5mm_P2.54mm_Vertical, Resistor_THT:R_Axial_DIN0207_L6.3mm_D2.5mm_P2.54mm_Vertical, F.Cu at (324.7, 277.5)
- added R7: R_Axial_DIN0207_L6.3mm_D2.5mm_P2.54mm_Vertical, Resistor_THT:R_Axial_DIN0207_L6.3mm_D2.5mm_P2.54mm_Vertical, F.Cu at (320.9, 277.5)
- added R74*: R_Axial_DIN0207_L6.3mm_D2.5mm_P2.54mm_Vertical, Resistor_THT:R_Axial_DIN0207_L6.3mm_D2.5mm_P2.54mm_Vertical, F.Cu at (305.6, 277.5)
- added R79: R_Axial_DIN0207_L6.3mm_D2.5mm_P2.54mm_Vertical, Resistor_THT:R_Axial_DIN0207_L6.3mm_D2.5mm_P2.54mm_Vertical, F.Cu at (137.3, 170.9)
- added R8: R_Axial_DIN0207_L6.3mm_D2.5mm_P2.54mm_Vertical, Resistor_THT:R_Axial_DIN0207_L6.3mm_D2.5mm_P2.54mm_Vertical, F.Cu at (317.1, 277.5)
- added R9: R_Axial_DIN0207_L6.3mm_D2.5mm_P2.54mm_Vertical, Resistor_THT:R_Axial_DIN0207_L6.3mm_D2.5mm_P2.54mm_Vertical, F.Cu at (309.5, 277.5)
- C11, C12, C13, C32, C33, C35, C36, C37, C38, C39, C40, C41, C42, C43, C44, C45, C46, C47, C48, C49, C50, C52, C53, C54, C55, C58, C59, C66, C67, C69, C7: footprint Capacitor_THT:C_Rect_L10.0mm_W3.0mm_P7.50mm_FKS3_FKP3 -> OSI:C_Rect_L10.0mm_W3.0mm_P7.50mm_FKS3_FKP3
Routing:
- net (no net): track 62585.1 -> 62580.1 mm, vias 2125 -> 2052
Other:
- board text removed: "C10"
- board text removed: "C12"
- board text removed: "C21"
- board text removed: "C22"
- board text removed: "C23"
- board text removed: "C24"
- board text removed: "C25"
- board text removed: "C26"
- board text removed: "C27"
- board text removed: "C28"
- board text removed: "C29"
- board text removed: "C30"
- board text removed: "C51"
- board text removed: "C56"
- board text removed: "C57"
- board text removed: "C6"
- board text removed: "C60"
- board text removed: "C61"
- board text removed: "C62"
- board text removed: "C65"
- board text removed: "C68"
- board text removed: "C8"
- board text removed: "F1"
- board text removed: "R10"
- board text removed: "R11"
- board text removed: "R2"
- board text removed: "R3"
- board text removed: "R4"
- board text removed: "R5"
- board text removed: "R6"
- board text removed: "R7"
- board text removed: "R74*"
- board text removed: "R8"
- board text removed: "R9"

Commit message: more footprints
Parts:
- removed the ? at (132.5, 170.0)
- added LED1: LED_D5.0mm, LED_THT:LED_D5.0mm, F.Cu at (131.0, 168.3)
- added U59: DIP-16_W7.62mm_LongPads, Package_DIP:DIP-16_W7.62mm_LongPads, F.Cu at (251.4, 96.4)
- added U60: DIP-16_W7.62mm_LongPads, Package_DIP:DIP-16_W7.62mm_LongPads, F.Cu at (232.4, 96.5)
- added U61: DIP-16_W7.62mm_LongPads, Package_DIP:DIP-16_W7.62mm_LongPads, F.Cu at (213.3, 96.4)
- added U64: DIP-16_W7.62mm_LongPads, Package_DIP:DIP-16_W7.62mm_LongPads, F.Cu at (156.3, 96.4)
- added U65: DIP-16_W7.62mm_LongPads, Package_DIP:DIP-16_W7.62mm_LongPads, F.Cu at (137.4, 96.4)
- added U66: DIP-8_W7.62mm_LongPads, Package_DIP:DIP-8_W7.62mm_LongPads, F.Cu at (232.4, 59.6)
- added U67: 7803, Package_DIP:DIP-14_W7.62mm_LongPads, F.Cu at (213.5, 63.4)
- added U68: 7803, Package_DIP:DIP-14_W7.62mm_LongPads, F.Cu at (194.4, 63.4)
- added U69: DIP-16_W7.62mm_LongPads, Package_DIP:DIP-16_W7.62mm_LongPads, F.Cu at (175.4, 63.4)
- added U80: DIP-8_W7.62mm_LongPads, Package_DIP:DIP-8_W7.62mm_LongPads, F.Cu at (137.6, 320.8)
- moved C12 0.10 mm to (225.0, 63.0)
Routing:
- net (no net): track 62580.1 -> 62197.9 mm, vias 2052 -> 1918
Other:
- board text removed: "LED1"
- board text removed: "U59"
- board text removed: "U60"
- board text removed: "U61"
- board text removed: "U64"
- board text removed: "U65"
- board text removed: "U66"
- board text removed: "U67"
- board text removed: "U68"
- board text removed: "U69"
- board text removed: "U80"
