File: src/OSI 600D Superboard II Cherry Solder Mask.kicad_pcb (KiCad board)
At the start: 2 copper layers, 301.5 x 367.3 mm, 182 parts, among them J2 CONN_SDA-41815_12_RA_MOL, J3 CONN_SDA-41815_12_RA_MOL, SW1 SW_Cherry_MX_1.00u_PCB, SW2 SW_Cherry_MX_1.00u_PCB, U41 CHR ROM, U59 DIP-16_W7.62mm_LongPads, U60 DIP-16_W7.62mm_LongPads, U61 DIP-16_W7.62mm_LongPads, U64 DIP-16_W7.62mm_LongPads, U65 DIP-16_W7.62mm_LongPads, U66 DIP-8_W7.62mm_LongPads, U67 7803, U68 7803, U69 DIP-16_W7.62mm_LongPads, U70 7803, U8 6502, U80 DIP-8_W7.62mm_LongPads

Commit message: more footprints and some nets added
Parts:
- added U14: 27C16 / 2816, Package_DIP:DIP-24_W15.24mm_LongPads, F.Cu at (153.6, 271.3)
- added U18: 7803, Package_DIP:DIP-14_W7.62mm_LongPads, F.Cu at (156.4, 228.1)
- added U19: 7803, Package_DIP:DIP-14_W7.62mm_LongPads, F.Cu at (137.3, 228.1)
- added U2: DIP-16_W7.62mm_LongPads, Package_DIP:DIP-16_W7.62mm_LongPads, F.Cu at (362.9, 271.3)
- added U3: DIP-16_W7.62mm_LongPads, Package_DIP:DIP-16_W7.62mm_LongPads, F.Cu at (362.8, 246.1)
- added U31: 2114, Package_DIP:DIP-18_W7.62mm_LongPads, F.Cu at (391.0, 162.5)
- added U32: 2114, Package_DIP:DIP-18_W7.62mm_LongPads, F.Cu at (374.4, 162.5)
- added U33: 2114, Package_DIP:DIP-18_W7.62mm_LongPads, F.Cu at (357.9, 162.5)
- added U34: 2114, Package_DIP:DIP-18_W7.62mm_LongPads, F.Cu at (341.4, 162.5)
- added U35: 2114, Package_DIP:DIP-18_W7.62mm_LongPads, F.Cu at (324.9, 162.4)
- added U36: 2114, Package_DIP:DIP-18_W7.62mm_LongPads, F.Cu at (308.5, 162.5)
- added U37: 2114, Package_DIP:DIP-18_W7.62mm_LongPads, F.Cu at (292.0, 162.5)
- added U38: 2114, Package_DIP:DIP-18_W7.62mm_LongPads, F.Cu at (275.5, 162.5)
- added U4: 7803, Package_DIP:DIP-14_W7.62mm_LongPads, F.Cu at (340.0, 271.3)
- added U42: DIP-16_W7.62mm_LongPads, Package_DIP:DIP-16_W7.62mm_LongPads, F.Cu at (175.4, 162.5)
- added U45: 2114, Package_DIP:DIP-18_W7.62mm_LongPads, F.Cu at (391.0, 129.5)
- added U46: 2114, Package_DIP:DIP-18_W7.62mm_LongPads, F.Cu at (374.5, 129.5)
- added U47: 2114, Package_DIP:DIP-18_W7.62mm_LongPads, F.Cu at (357.9, 129.5)
- added U48: 2114, Package_DIP:DIP-18_W7.62mm_LongPads, F.Cu at (341.4, 129.5)
- added U49: 2114, Package_DIP:DIP-18_W7.62mm_LongPads, F.Cu at (325.0, 129.5)
- added U5: 7803, Package_DIP:DIP-14_W7.62mm_LongPads, F.Cu at (340.1, 246.1)
- added U50: 2114, Package_DIP:DIP-18_W7.62mm_LongPads, F.Cu at (308.6, 129.5)
- added U51: 2114, Package_DIP:DIP-18_W7.62mm_LongPads, F.Cu at (292.0, 129.5)
- added U52: 2114, Package_DIP:DIP-18_W7.62mm_LongPads, F.Cu at (275.6, 129.5)
- added U53: DIP-16_W7.62mm_LongPads, Package_DIP:DIP-16_W7.62mm_LongPads, F.Cu at (251.3, 129.5)
- added U54: DIP-16_W7.62mm_LongPads, Package_DIP:DIP-16_W7.62mm_LongPads, F.Cu at (232.4, 129.5)
- added U57: DIP-16_W7.62mm_LongPads, Package_DIP:DIP-16_W7.62mm_LongPads, F.Cu at (175.5, 129.5)
- added U58: 7803, Package_DIP:DIP-14_W7.62mm_LongPads, F.Cu at (156.3, 129.5)
- added U6: DIP-16_W7.62mm_LongPads, Package_DIP:DIP-16_W7.62mm_LongPads, F.Cu at (317.1, 271.3)
- added U7: DIP-16_W7.62mm_LongPads, Package_DIP:DIP-16_W7.62mm_LongPads, F.Cu at (317.1, 246.1)
- moved G*** 73.9 mm to (288.4, 97.5)
Routing:
- net (no net): track 62197.9 -> 33256.7 mm, vias 1918 -> 916
- net GND: track 0.00 -> 8904.7 mm, vias 0 -> 149
- net Vcc: track 0.00 -> 5464.8 mm, vias 0 -> 123
- net A6: track 0.00 -> 1175.2 mm, vias 0 -> 22
- net A0: track 0.00 -> 1143.6 mm, vias 0 -> 24
- net D1: track 0.00 -> 1021.9 mm, vias 0 -> 20
- net A3: track 0.00 -> 967.7 mm, vias 0 -> 11
- net A8: track 0.00 -> 877.7 mm, vias 0 -> 17
- net A9: track 0.00 -> 838.7 mm, vias 0 -> 16
- net A7: track 0.00 -> 838.6 mm, vias 0 -> 13
- net /~{WE}: track 0.00 -> 818.2 mm, vias 0 -> 8
- net A2: track 0.00 -> 801.1 mm, vias 0 -> 11
- net A4: track 0.00 -> 758.2 mm, vias 0 -> 12
- net A5: track 0.00 -> 744.1 mm, vias 0 -> 13
- net A1: track 0.00 -> 741.7 mm, vias 0 -> 11
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Other:
- board text removed: "Bambelweeny57"
- board text removed: "U14"
- board text removed: "U18"
- board text removed: "U19"
- board text removed: "U2"
- board text removed: "U3"
- board text removed: "U31"
- board text removed: "U32"
- board text removed: "U33"
- board text removed: "U34"
- board text removed: "U35"
- board text removed: "U36"
- board text removed: "U37"
- board text removed: "U38"
- board text removed: "U4"
- board text removed: "U42"
- board text removed: "U45"
- board text removed: "U46"
- board text removed: "U47"
- board text removed: "U49"
- board text removed: "U5"
- board text removed: "U50"
- board text removed: "U51"
- board text removed: "U52"
- board text removed: "U53"
- board text removed: "U54"
- board text removed: "U57"
- board text removed: "U58"
- board text removed: "U6"
- board text removed: "U7"

Commit message: added io nets for ram
Connections:
- net D3 renamed IO4
- U52 pad 12: D2 -> IO3
- U52 pad 13: D1 -> IO2
- U52 pad 14: D0 -> IO1
Routing:
- net IO3: track 0.00 -> 641.3 mm, vias 0 -> 10
- net D2: track 641.3 -> 0.00 mm, vias 10 -> 0
- net IO1: track 0.00 -> 625.0 mm, vias 0 -> 11
- net D0: track 682.2 -> 57.1 mm, vias 13 -> 2
- net D1: track 1021.9 -> 400.7 mm, vias 20 -> 9
- net IO2: track 0.00 -> 621.2 mm, vias 0 -> 11

Commit message: more footprints
Parts:
- added U00: 7803, Package_DIP:DIP-14_W7.62mm_LongPads, F.Cu at (95.0, 217.8)
- added U00: DIP-16_W7.62mm_LongPads, Package_DIP:DIP-16_W7.62mm_LongPads, F.Cu at (95.0, 191.5)
- added U10: 27C16 / 2816, Package_DIP:DIP-24_W15.24mm_LongPads, F.Cu at (244.9, 271.3)
- added U11: 27C16 / 2816, Package_DIP:DIP-24_W15.24mm_LongPads, F.Cu at (222.2, 271.3)
- added U12: 27C16 / 2816, Package_DIP:DIP-24_W15.24mm_LongPads, F.Cu at (199.3, 271.3)
- added U13: 27C16 / 2816, Package_DIP:DIP-24_W15.24mm_LongPads, F.Cu at (176.4, 271.3)
- added U20: DIP-16_W7.62mm_LongPads, Package_DIP:DIP-16_W7.62mm_LongPads, F.Cu at (384.7, 195.3)
- added U21: 7803, Package_DIP:DIP-14_W7.62mm_LongPads, F.Cu at (365.7, 195.3)
- added U22: DIP-16_W7.62mm_LongPads, Package_DIP:DIP-16_W7.62mm_LongPads, F.Cu at (346.5, 195.3)
- added U23: DIP-16_W7.62mm_LongPads, Package_DIP:DIP-16_W7.62mm_LongPads, F.Cu at (327.4, 195.3)
- added U30: DIP-16_W7.62mm_LongPads, Package_DIP:DIP-16_W7.62mm_LongPads, F.Cu at (137.4, 195.4)
- added U39: 2114, Package_DIP:DIP-18_W7.62mm_LongPads, F.Cu at (242.4, 162.4)
- added U40: 2114, Package_DIP:DIP-18_W7.62mm_LongPads, F.Cu at (227.6, 162.4)
- added U62: 7803, Package_DIP:DIP-14_W7.62mm_LongPads, F.Cu at (194.4, 96.4)
- added U63: 7803, Package_DIP:DIP-14_W7.62mm_LongPads, F.Cu at (175.5, 96.4)
- added U77: 2114, Package_DIP:DIP-18_W7.62mm_LongPads, F.Cu at (256.3, 162.6)
- added U9: 27C16 / 2816, Package_DIP:DIP-24_W15.24mm_LongPads, F.Cu at (267.7, 271.3)
Connections:
- U14 pad 1: GND -> (no net)
- U14 pad 10: D1 -> (no net)
- U14 pad 11: D2 -> (no net)
- U14 pad 12: GND -> (no net)
- U14 pad 2: A6 -> (no net)
- U14 pad 23: W3-A8 -> (no net)
- U14 pad 24: Vcc -> (no net)
- U14 pad 3: W5-A5 -> (no net)
- U14 pad 4: W5-A4 -> (no net)
- U14 pad 8: A0 -> (no net)
- U14 pad 9: D0 -> (no net)
- U31 pad 18: Vcc -> (no net)
- U31 pad 9: GND -> (no net)
- U32 pad 18: Vcc -> (no net)
- U32 pad 9: GND -> (no net)
- U33 pad 18: Vcc -> (no net)
- U33 pad 9: GND -> (no net)
- U34 pad 18: Vcc -> (no net)
- U34 pad 9: GND -> (no net)
- U35 pad 18: Vcc -> (no net)
- U35 pad 9: GND -> (no net)
- U36 pad 18: Vcc -> (no net)
- U36 pad 9: GND -> (no net)
- U37 pad 18: Vcc -> (no net)
- U37 pad 9: GND -> (no net)
- U38 pad 18: Vcc -> (no net)
- U38 pad 9: GND -> (no net)
- U45 pad 18: Vcc -> (no net)
- U45 pad 9: GND -> (no net)
- U46 pad 18: Vcc -> (no net)
- U46 pad 9: GND -> (no net)
- U47 pad 18: Vcc -> (no net)
- U48 pad 18: Vcc -> (no net)
- U48 pad 9: GND -> (no net)
- U49 pad 18: Vcc -> (no net)
- U49 pad 9: GND -> (no net)
- U50 pad 18: Vcc -> (no net)
- U50 pad 9: GND -> (no net)
- U51 pad 18: Vcc -> (no net)
- U51 pad 9: GND -> (no net)
- U52 pad 1: A6 -> (no net)
- U52 pad 10: /~{WE} -> (no net)
- U52 pad 11: IO4 -> (no net)
- U52 pad 12: IO3 -> (no net)
- U52 pad 13: IO2 -> (no net)
- U52 pad 14: IO1 -> (no net)
- U52 pad 15: A9 -> (no net)
- U52 pad 16: A8 -> (no net)
- U52 pad 17: A7 -> (no net)
- U52 pad 18: Vcc -> (no net)
- U52 pad 2: A5 -> (no net)
- U52 pad 3: A4 -> (no net)
- U52 pad 4: A3 -> (no net)
- U52 pad 5: A0 -> (no net)
- U52 pad 6: A1 -> (no net)
- U52 pad 7: A2 -> (no net)
- U52 pad 8: /~{CS} -> (no net)
- U52 pad 9: GND -> (no net)
Routing:
- net (no net): track 33256.7 -> 59916.0 mm, vias 916 -> 1128
- net GND: track 8904.7 -> 0.00 mm, vias 149 -> 0
- net Vcc: track 5464.8 -> 0.00 mm, vias 123 -> 0
- net A6: track 1175.2 -> 0.00 mm, vias 22 -> 0
- net A0: track 1143.6 -> 0.00 mm, vias 24 -> 0
- net A3: track 967.7 -> 0.00 mm, vias 11 -> 0
- net A8: track 877.7 -> 0.00 mm, vias 17 -> 0
- net A9: track 838.7 -> 0.00 mm, vias 16 -> 0
- net A7: track 838.6 -> 0.00 mm, vias 13 -> 0
- net /~{WE}: track 818.2 -> 0.00 mm, vias 8 -> 0
- net A2: track 801.1 -> 0.00 mm, vias 11 -> 0
- net A4: track 758.2 -> 0.00 mm, vias 12 -> 0
- net A5: track 744.1 -> 0.00 mm, vias 13 -> 0
- net A1: track 741.7 -> 0.00 mm, vias 11 -> 0
- net IO4: track 643.9 -> 0.00 mm, vias 10 -> 0
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Other:
- board text removed: "R1"
- board text removed: "U10"
- board text removed: "U11"
- board text removed: "U12"
- board text removed: "U13"
- board text removed: "U20"
- board text removed: "U21"
- board text removed: "U22"
- board text removed: "U23"
- board text removed: "U30"
- board text removed: "U39"
- board text removed: "U40"
- board text removed: "U62"
- board text removed: "U63"
- board text removed: "U77"
- board text removed: "U9"
