File: src/OSI 600D Superboard II Cherry Solder Mask.kicad_pcb (KiCad board)
At the start: 2 copper layers, 301.5 x 367.3 mm, 229 parts, among them J2 CONN_SDA-41815_12_RA_MOL, J3 CONN_SDA-41815_12_RA_MOL, SW1 SW_Cherry_MX_1.00u_PCB, SW2 SW_Cherry_MX_1.00u_PCB, U00 7803, U00 DIP-16_W7.62mm_LongPads, U10 27C16 / 2816, U11 27C16 / 2816, U12 27C16 / 2816, U13 27C16 / 2816, U14 27C16 / 2816, U18 7803, U19 7803, U2 DIP-16_W7.62mm_LongPads, U20 DIP-16_W7.62mm_LongPads, U21 7803, U22 DIP-16_W7.62mm_LongPads, U23 DIP-16_W7.62mm_LongPads, U3 DIP-16_W7.62mm_LongPads, U30 DIP-16_W7.62mm_LongPads, U31 2114, U32 2114, U33 2114, U34 2114, U35 2114, U36 2114, U37 2114, U38 2114, U39 2114, U4 7803, U40 2114, U41 CHR ROM, U42 DIP-16_W7.62mm_LongPads, U45 2114, U46 2114, U47 2114, U48 2114, U49 2114, U5 7803, U50 2114, U51 2114, U52 2114, U53 DIP-16_W7.62mm_LongPads, U54 DIP-16_W7.62mm_LongPads, U57 DIP-16_W7.62mm_LongPads, U58 7803, U59 DIP-16_W7.62mm_LongPads, U6 DIP-16_W7.62mm_LongPads, U60 DIP-16_W7.62mm_LongPads, U61 DIP-16_W7.62mm_LongPads, U62 7803, U63 7803, U64 DIP-16_W7.62mm_LongPads, U65 DIP-16_W7.62mm_LongPads, U66 DIP-8_W7.62mm_LongPads, U67 7803, U68 7803, U69 DIP-16_W7.62mm_LongPads, U7 DIP-16_W7.62mm_LongPads, U70 7803, U77 2114, U8 6502, U80 DIP-8_W7.62mm_LongPads, U9 27C16 / 2816

Commit message: more footprints
Parts:
- removed U00: 7803, Package_DIP:DIP-14_W7.62mm_LongPads
- removed U00: DIP-16_W7.62mm_LongPads, Package_DIP:DIP-16_W7.62mm_LongPads
- added D17: D_DO-34_SOD68_P10.16mm_Horizontal, Diode_THT:D_DO-34_SOD68_P10.16mm_Horizontal, F.Cu at (389.1, 373.0)
- added D18: D_DO-34_SOD68_P10.16mm_Horizontal, Diode_THT:D_DO-34_SOD68_P10.16mm_Horizontal, F.Cu at (391.8, 373.0)
- added D19: D_DO-34_SOD68_P10.16mm_Horizontal, Diode_THT:D_DO-34_SOD68_P10.16mm_Horizontal, F.Cu at (394.4, 373.0)
- added D20: D_DO-34_SOD68_P10.16mm_Horizontal, Diode_THT:D_DO-34_SOD68_P10.16mm_Horizontal, F.Cu at (396.9, 373.0)
- added D21: D_DO-34_SOD68_P10.16mm_Horizontal, Diode_THT:D_DO-34_SOD68_P10.16mm_Horizontal, F.Cu at (399.5, 373.0)
- added D22: D_DO-34_SOD68_P10.16mm_Horizontal, Diode_THT:D_DO-34_SOD68_P10.16mm_Horizontal, F.Cu at (402.1, 373.0)
- added D23: D_DO-34_SOD68_P10.16mm_Horizontal, Diode_THT:D_DO-34_SOD68_P10.16mm_Horizontal, F.Cu at (404.5, 373.0)
- added D24: D_DO-34_SOD68_P10.16mm_Horizontal, Diode_THT:D_DO-34_SOD68_P10.16mm_Horizontal, F.Cu at (406.9, 373.0)
- added J1: 6502, Package_DIP:DIP-40_W15.24mm_LongPads, F.Cu at (378.3, 223.3)
- added J75: DIP-16_W7.62mm_LongPads, Package_DIP:DIP-16_W7.62mm_LongPads, F.Cu at (200.5, 177.7)
- added R37: R_Yageo_L3.6mm_D1.6mm_P12.70mm_Horizontal, Mod:R_Yageo_L3.6mm_D1.6mm_P12.70mm_Horizontal, F.Cu at (222.3, 43.2)
- added R77: R_Yageo_L3.6mm_D1.6mm_P12.70mm_Horizontal, Mod:R_Yageo_L3.6mm_D1.6mm_P12.70mm_Horizontal, F.Cu at (130.9, 328.1)
- added R78: R_Yageo_L3.6mm_D1.6mm_P12.70mm_Horizontal, Mod:R_Yageo_L3.6mm_D1.6mm_P12.70mm_Horizontal, F.Cu at (130.9, 331.2)
- added R79: R_Yageo_L3.6mm_D1.6mm_P12.70mm_Horizontal, Mod:R_Yageo_L3.6mm_D1.6mm_P12.70mm_Horizontal, F.Cu at (131.0, 334.5)
- added R80: R_Yageo_L3.6mm_D1.6mm_P12.70mm_Horizontal, Mod:R_Yageo_L3.6mm_D1.6mm_P12.70mm_Horizontal, F.Cu at (130.9, 337.5)
- added R81: R_Yageo_L3.6mm_D1.6mm_P12.70mm_Horizontal, Mod:R_Yageo_L3.6mm_D1.6mm_P12.70mm_Horizontal, F.Cu at (130.9, 340.7)
- added R82: R_Yageo_L3.6mm_D1.6mm_P12.70mm_Horizontal, Mod:R_Yageo_L3.6mm_D1.6mm_P12.70mm_Horizontal, F.Cu at (130.9, 344.1)
- added R83: R_Yageo_L3.6mm_D1.6mm_P12.70mm_Horizontal, Mod:R_Yageo_L3.6mm_D1.6mm_P12.70mm_Horizontal, F.Cu at (130.9, 347.1)
- added R84: R_Yageo_L3.6mm_D1.6mm_P12.70mm_Horizontal, Mod:R_Yageo_L3.6mm_D1.6mm_P12.70mm_Horizontal, F.Cu at (130.9, 350.3)
- added R85: R_Yageo_L3.6mm_D1.6mm_P12.70mm_Horizontal, Mod:R_Yageo_L3.6mm_D1.6mm_P12.70mm_Horizontal, F.Cu at (149.2, 371.1)
- added U15: 7803, Package_DIP:DIP-14_W7.62mm_LongPads, F.Cu at (228.9, 228.0)
- added U16: 7803, Package_DIP:DIP-14_W7.62mm_LongPads, F.Cu at (212.9, 228.2)
- added U17: DIP-16_W7.62mm_LongPads, Package_DIP:DIP-16_W7.62mm_LongPads, F.Cu at (179.6, 228.4)
- added U24: DIP-16_W7.62mm_LongPads, Package_DIP:DIP-16_W7.62mm_LongPads, F.Cu at (240.9, 195.3)
- added U25: DIP-16_W7.62mm_LongPads, Package_DIP:DIP-16_W7.62mm_LongPads, F.Cu at (225.4, 195.4)
- added U29: 7803, Package_DIP:DIP-14_W7.62mm_LongPads, F.Cu at (156.5, 195.2)
- added U43: 7803, Package_DIP:DIP-14_W7.62mm_LongPads, F.Cu at (190.7, 195.3)
- added U55: DIP-16_W7.62mm_LongPads, Package_DIP:DIP-16_W7.62mm_LongPads, F.Cu at (213.3, 129.5)
- added U56: 7803, Package_DIP:DIP-14_W7.62mm_LongPads, F.Cu at (194.7, 129.5)
- added U72: DIP-16_W7.62mm_LongPads, Package_DIP:DIP-16_W7.62mm_LongPads, F.Cu at (245.7, 230.7)
- added U73: DIP-16_W7.62mm_LongPads, Package_DIP:DIP-16_W7.62mm_LongPads, F.Cu at (197.0, 228.2)
- added U74: DIP-16_W7.62mm_LongPads, Package_DIP:DIP-16_W7.62mm_LongPads, F.Cu at (256.1, 195.3)
- added U76: 7803, Package_DIP:DIP-14_W7.62mm_LongPads, F.Cu at (173.9, 195.3)
- added U78: DIP-16_W7.62mm_LongPads, Package_DIP:DIP-16_W7.62mm_LongPads, F.Cu at (155.2, 162.5)
- added U79: 7803, Package_DIP:DIP-14_W7.62mm_LongPads, F.Cu at (137.7, 162.3)
Routing:
- net (no net): track 59916.0 -> 59467.2 mm, vias 1128 -> 810
Other:
- board text removed: "D17"
- board text removed: "D18"
- board text removed: "D19"
- board text removed: "D20"
- board text removed: "D21"
- board text removed: "D22"
- board text removed: "D23"
- board text removed: "D24"
- board text removed: "J1"
- board text removed: "J75"
- board text removed: "R37"
- board text removed: "R76"
- board text removed: "R77"
- board text removed: "R78"
- board text removed: "R79"
- board text removed: "R80"
- board text removed: "R81"
- board text removed: "R82"
- board text removed: "R83"
- board text removed: "R84"
- board text removed: "R85"
- board text removed: "U15"
- board text removed: "U16"
- board text removed: "U17"
- board text removed: "U24"
- board text removed: "U25"
- board text removed: "U29"
- board text removed: "U43"
- board text removed: "U55"
- board text removed: "U56"
- board text removed: "U72"
- board text removed: "U73"
- board text removed: "U74"
- board text removed: "U76"
- board text removed: "U78"
- board text removed: "U79"

Commit message: more foot prints
Parts:
- added C5: CP_Axial_L10.0mm_D4.5mm_P15.00mm_Horizontal, Capacitor_THT:CP_Axial_L10.0mm_D4.5mm_P15.00mm_Horizontal, F.Cu at (267.8, 61.5)
- added D1: D_DO-34_SOD68_P10.16mm_Horizontal, Diode_THT:D_DO-34_SOD68_P10.16mm_Horizontal, F.Cu at (365.2, 277.4)
- added D10: D_DO-34_SOD68_P10.16mm_Horizontal, Diode_THT:D_DO-34_SOD68_P10.16mm_Horizontal, F.Cu at (233.8, 48.3)
- added D15: D_DO-35_SOD27_P12.70mm_Horizontal, Diode_THT:D_DO-35_SOD27_P12.70mm_Horizontal, F.Cu at (262.9, 100.3)
- added D2: D_DO-34_SOD68_P10.16mm_Horizontal, Diode_THT:D_DO-34_SOD68_P10.16mm_Horizontal, F.Cu at (362.8, 277.4)
- added D25: D_DO-34_SOD68_P10.16mm_Horizontal, Diode_THT:D_DO-34_SOD68_P10.16mm_Horizontal, F.Cu at (152.4, 306.6)
- added D26: D_DO-34_SOD68_P10.16mm_Horizontal, Diode_THT:D_DO-34_SOD68_P10.16mm_Horizontal, F.Cu at (152.4, 309.2)
- added D27: D_DO-34_SOD68_P10.16mm_Horizontal, Diode_THT:D_DO-34_SOD68_P10.16mm_Horizontal, F.Cu at (146.0, 361.2)
- added D29: D_DO-34_SOD68_P10.16mm_Horizontal, Diode_THT:D_DO-34_SOD68_P10.16mm_Horizontal, F.Cu at (149.2, 378.6)
- added D3: D_DO-34_SOD68_P10.16mm_Horizontal, Diode_THT:D_DO-34_SOD68_P10.16mm_Horizontal, F.Cu at (360.2, 277.4)
- added D30: D_DO-34_SOD68_P10.16mm_Horizontal, Diode_THT:D_DO-34_SOD68_P10.16mm_Horizontal, F.Cu at (140.9, 353.3)
- added D31: D_DO-34_SOD68_P10.16mm_Horizontal, Diode_THT:D_DO-34_SOD68_P10.16mm_Horizontal, F.Cu at (140.9, 356.8)
- added D32: D_DO-34_SOD68_P10.16mm_Horizontal, Diode_THT:D_DO-34_SOD68_P10.16mm_Horizontal, F.Cu at (139.6, 299.1)
- added D4: D_DO-34_SOD68_P10.16mm_Horizontal, Diode_THT:D_DO-34_SOD68_P10.16mm_Horizontal, F.Cu at (357.6, 277.4)
- added D5: D_DO-34_SOD68_P10.16mm_Horizontal, Diode_THT:D_DO-34_SOD68_P10.16mm_Horizontal, F.Cu at (355.2, 277.4)
- added D6: D_DO-34_SOD68_P10.16mm_Horizontal, Diode_THT:D_DO-34_SOD68_P10.16mm_Horizontal, F.Cu at (352.5, 277.4)
- added D7: D_DO-34_SOD68_P10.16mm_Horizontal, Diode_THT:D_DO-34_SOD68_P10.16mm_Horizontal, F.Cu at (350.0, 277.4)
- added D8: D_DO-34_SOD68_P10.16mm_Horizontal, Diode_THT:D_DO-34_SOD68_P10.16mm_Horizontal, F.Cu at (347.5, 277.4)
- added D9: D_DO-34_SOD68_P10.16mm_Horizontal, Diode_THT:D_DO-34_SOD68_P10.16mm_Horizontal, F.Cu at (233.8, 45.8)
- added R64: 1K, Mod:R_Axial_DIN0516_L15.5mm_D5.0mm_P22.60mm_Horizontal, F.Cu at (245.4, 48.7)
- added R65: R_Axial_DIN0309_L9.0mm_D3.2mm_P20.32mm_Horizontal, Resistor_THT:R_Axial_DIN0309_L9.0mm_D3.2mm_P20.32mm_Horizontal, F.Cu at (278.4, 93.4)
- added R76: R_Yageo_L3.6mm_D1.6mm_P12.70mm_Horizontal, Mod:R_Yageo_L3.6mm_D1.6mm_P12.70mm_Horizontal, F.Cu at (130.8, 325.0)
Routing:
- net (no net): track 59467.2 -> 59521.1 mm, vias 810 -> 759
Other:
- board text removed: "C5"
- board text removed: "D1"
- board text removed: "D10"
- board text removed: "D15"
- board text removed: "D2"
- board text removed: "D25"
- board text removed: "D26"
- board text removed: "D27"
- board text removed: "D29"
- board text removed: "D3"
- board text removed: "D30"
- board text removed: "D31"
- board text removed: "D32"
- board text removed: "D4"
- board text removed: "D5"
- board text removed: "D6"
- board text removed: "D7"
- board text removed: "D8"
- board text removed: "D9"
- board text removed: "R64"
- board text removed: "R65"

Commit message: added values to known ic's
Parts:
- C5: value CP_Axial_L10.0mm_D4.5mm_P15.00mm_Horizontal -> 47uf
- D15: value D_DO-35_SOD27_P12.70mm_Horizontal -> 1N4001
- J1: value 6502 -> DIP40
- J75: value DIP-16_W7.62mm_LongPads -> DIP16
- U15: value 7803 -> 74LS02
- U16, U18: value 7803 -> 74LS04
- U17: value DIP-16_W7.62mm_LongPads -> 74LS159
- U19, U56: value 7803 -> 74LS20
- U2, U3: value DIP-16_W7.62mm_LongPads -> 74LS75
- U24, U25, U74: value DIP-16_W7.62mm_LongPads -> 8T28
- U29, U43, U62: value 7803 -> ?
- U30, U57, U59, U60, U61: value DIP-16_W7.62mm_LongPads -> 74LS163
- U4, U5: value 7803 -> 74LS125
- U42: value DIP-16_W7.62mm_LongPads -> 74LS165
- U53, U55, U78: value DIP-16_W7.62mm_LongPads -> 74LS157
- U54: value DIP-16_W7.62mm_LongPads -> 74LS175
- U58: value 7803 -> 74LS00
- U6, U7: value DIP-16_W7.62mm_LongPads -> T828
- U63, U76: value 7803 -> 74LS74
- U64: value DIP-16_W7.62mm_LongPads -> 74LS76
- U65, U69: value DIP-16_W7.62mm_LongPads -> 74LS123
- U66, U80: value DIP-8_W7.62mm_LongPads -> ?
- U67: value 7803 -> 74LS14
- U68: value 7803 -> 74LS17
- U70: value 7803 -> 74LS03
- U72: value DIP-16_W7.62mm_LongPads -> 74LS174
- U73: value DIP-16_W7.62mm_LongPads -> 74LS138
- U79: value 7803 -> 74LS86
Changed lines of the file:
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@@
 			)
 		)
-		(property "Value" "DIP-8_W7.62mm_LongPads"
+		(property "Value" "?"
 			(at 3.81 9.95 0)
 			(layer "F.Fab")
@@
 			)
 		)
-		(property "Value" "DIP-16_W7.62mm_LongPads"
+		(property "Value" "74LS174"
 			(at 3.81 20.11 0)
 			(layer "F.Fab")
@@
 			)
 		)
-		(property "Value" "7803"
+		(property "Value" "?"
 			(at 3.81 17.57 0)
 			(layer "F.Fab")
@@
 			)
 		)
-		(property "Value" "7803"
+		(property "Value" "74LS02"
 			(at 3.81 17.57 0)
 			(layer "F.Fab")
@@
 			)
 		)
-		(property "Value" "7803"
+		(property "Value" "74LS20"
 			(at 3.81 17.57 0)
 			(layer "F.Fab")
@@
 			)
 		)
-		(property "Value" "7803"
+		(property "Value" "?"
 			(at 3.81 17.57 0)
 			(layer "F.Fab")
@@
 			)
 		)
-		(property "Value" "DIP-16_W7.62mm_LongPads"
+		(property "Value" "74LS75"
 			(at 3.81 20.11 0)
 			(layer "F.Fab")
@@
 			)
 		)
-		(property "Value" "DIP-16_W7.62mm_LongPads"
+		(property "Value" "74LS138"
 			(at 3.81 20.11 0)
 			(layer "F.Fab")
@@
 			)
 		)
-		(property "Value" "7803"
+		(property "Value" "?"
 			(at 3.81 17.57 0)
 			(layer "F.Fab")
@@
 			)
 		)
-		(property "Value" "6502"
+		(property "Value" "DIP40"
 			(at 7.62 50.59 0)
 			(layer "F.Fab")
@@
 			)
 		)
-		(property "Value" "7803"
+		(property "Value" "74LS00"
 			(at 3.81 17.57 0)
 			(layer "F.Fab")
@@
 			)
 		)
-		(property "Value" "7803"
+		(property "Value" "74LS14"
 			(at 3.81 17.57 0)
 			(layer "F.Fab")
@@
 			)
 		)
-		(property "Value" "DIP-16_W7.62mm_LongPads"
+		(property "Value" "74LS163"
 			(at 3.81 20.11 0)
 			(layer "F.Fab")
@@
 			)
 		)
-		(property "Value" "DIP-8_W7.62mm_LongPads"
+		(property "Value" "?"
 			(at 3.81 9.95 0)
 			(layer "F.Fab")
@@
 			)
 		)
-		(property "Value" "7803"
+		(property "Value" "74LS03"
 			(at 3.81 17.57 0)
 			(layer "F.Fab")
@@
 			)
 		)
-		(property "Value" "DIP-16_W7.62mm_LongPads"
+		(property "Value" "74LS123"
 			(at 3.81 20.11 0)
 			(layer "F.Fab")
@@
 			)
 		)
-		(property "Value" "DIP-16_W7.62mm_LongPads"
+		(property "Value" "74LS163"
 			(at 3.81 20.11 0)
 			(layer "F.Fab")
@@
 			)
 		)
-		(property "Value" "D_DO-35_SOD27_P12.70mm_Horizontal"
+		(property "Value" "1N4001"
 			(at 6.35 2.12 90)
 			(layer "F.Fab")
@@
 			)
 		)
-		(property "Value" "DIP-16_W7.62mm_LongPads"
+		(property "Value" "T828"
 			(at 3.81 20.11 0)
 			(layer "F.Fab")
@@
 			)
 		)
-		(property "Value" "DIP-16_W7.62mm_LongPads"
+		(property "Value" "8T28"
 			(at 3.81 20.11 0)
 			(layer "F.Fab")
@@
 			)
 		)
-		(property "Value" "DIP-16_W7.62mm_LongPads"
+		(property "Value" "74LS163"
 			(at 3.81 20.11 0)
 			(layer "F.Fab")
@@
 			)
 		)
-		(property "Value" "DIP-16_W7.62mm_LongPads"
+		(property "Value" "8T28"
 			(at 3.81 20.11 0)
 			(layer "F.Fab")
@@
 			)
 		)
-		(property "Value" "CP_Axial_L10.0mm_D4.5mm_P15.00mm_Horizontal"
+		(property "Value" "47uf"
 			(at 7.5 3.37 90)
 			(layer "F.Fab")
@@
 			)
 		)
-		(property "Value" "7803"
+		(property "Value" "74LS86"
 			(at 3.81 17.57 0)
 			(layer "F.Fab")
@@
 			)
 		)
-		(property "Value" "DIP-16_W7.62mm_LongPads"
+		(property "Value" "74LS123"
 			(at 3.81 20.11 0)
 			(layer "F.Fab")
@@
 			)
 		)
-		(property "Value" "DIP-16_W7.62mm_LongPads"
+		(property "Value" "DIP16"
 			(at 3.81 20.11 0)
 			(layer "F.Fab")
@@
 			)
 		)
-		(property "Value" "7803"
+		(property "Value" "74LS125"
 			(at 3.81 17.57 0)
 			(layer "F.Fab")
@@
 			)
 		)
-		(property "Value" "7803"
+		(property "Value" "74LS74"
 			(at 3.81 17.57 0)
 			(layer "F.Fab")
@@
 			)
 		)
-		(property "Value" "DIP-16_W7.62mm_LongPads"
+		(property "Value" "74LS159"
 			(at 3.81 20.11 0)
 			(layer "F.Fab")
@@
 			)
 		)
-		(property "Value" "7803"
+		(property "Value" "74LS74"
 			(at 3.81 17.57 0)
 			(layer "F.Fab")
@@
 			)
 		)
-		(property "Value" "DIP-16_W7.62mm_LongPads"
+		(property "Value" "8T28"
 			(at 3.81 20.11 0)
 			(layer "F.Fab")
@@
 			)
 		)
-		(property "Value" "DIP-16_W7.62mm_LongPads"
+		(property "Value" "74LS157"
 			(at 3.81 20.11 0)
 			(layer "F.Fab")
@@
 			)
 		)
-		(property "Value" "7803"
+		(property "Value" "74LS20"
 			(at 3.81 17.57 0)
 			(layer "F.Fab")
@@
 			)
 		)
-		(property "Value" "DIP-16_W7.62mm_LongPads"
+		(property "Value" "74LS76"
 			(at 3.81 20.11 0)
 			(layer "F.Fab")
@@
 			)
 		)
-		(property "Value" "7803"
+		(property "Value" "74LS04"
 			(at 3.81 17.57 0)
 			(layer "F.Fab")
@@
 			)
 		)
-		(property "Value" "DIP-16_W7.62mm_LongPads"
+		(property "Value" "T828"
 			(at 3.81 20.11 0)
 			(layer "F.Fab")
@@
 			)
 		)
-		(property "Value" "DIP-16_W7.62mm_LongPads"
+		(property "Value" "74LS157"
 			(at 3.81 20.11 0)
 			(layer "F.Fab")
@@
 			)
 		)
-		(property "Value" "DIP-16_W7.62mm_LongPads"
+		(property "Value" "74LS163"
 			(at 3.81 20.11 0)
 			(layer "F.Fab")
@@
 			)
 		)
-		(property "Value" "DIP-16_W7.62mm_LongPads"
+		(property "Value" "74LS163"
 			(at 3.81 20.11 0)
 			(layer "F.Fab")
@@
 			)
 		)
-		(property "Value" "7803"
+		(property "Value" "74LS17"
 			(at 3.81 17.57 0)
 			(layer "F.Fab")
@@
 			)
 		)
-		(property "Value" "DIP-16_W7.62mm_LongPads"
+		(property "Value" "74LS165"
 			(at 3.81 20.11 0)
 			(layer "F.Fab")
@@
 			)
 		)
-		(property "Value" "DIP-16_W7.62mm_LongPads"
+		(property "Value" "74LS175"
 			(at 3.81 20.11 0)
 			(layer "F.Fab")
@@
 			)
 		)
-		(property "Value" "7803"
+		(property "Value" "74LS125"
 			(at 3.81 17.57 0)
 			(layer "F.Fab")
@@
 			)
 		)
-		(property "Value" "7803"
+		(property "Value" "74LS04"
 			(at 3.81 17.57 0)
 			(layer "F.Fab")
@@
 			)
 		)
-		(property "Value" "DIP-16_W7.62mm_LongPads"
+		(property "Value" "74LS75"
 			(at 3.81 20.11 0)
 			(layer "F.Fab")
@@
 			)
 		)
-		(property "Value" "DIP-16_W7.62mm_LongPads"
+		(property "Value" "74LS157"
 			(at 3.81 20.11 0)
 			(layer "F.Fab")
