File: src/OSI 600D Superboard II Cherry Solder Mask - Copy.kicad_pcb (KiCad board)
At the start: 2 copper layers, 301.5 x 367.3 mm, 293 parts, among them J1 DIP40, J2 CONN_SDA-41815_12_RA_MOL, J3 CONN_SDA-41815_12_RA_MOL, J4 Molex_KK-396_A-41791-0002_1x0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, J75 DIP16, Q1 TO-92L_Wide, Q2 TO-92L_Wide, SW1 SW_Cherry_MX_1.00u_PCB, SW10 SW_Cherry_MX_1.00u_PCB, SW11 SW_Cherry_MX_1.00u_PCB, SW12 SW_Cherry_MX_1.00u_PCB, SW13 SW_Cherry_MX_1.00u_PCB, SW14 SW_Cherry_MX_1.00u_PCB, SW15 SW_Cherry_MX_1.00u_PCB, SW16 SW_Cherry_MX_1.00u_PCB, SW17 SW_Cherry_MX_1.00u_PCB, SW18 SW_Cherry_MX_1.00u_PCB, SW19 SW_Cherry_MX_1.00u_PCB, SW2 SW_Cherry_MX_1.00u_PCB, SW20 SW_Cherry_MX_1.00u_PCB, SW21 SW_Cherry_MX_1.00u_PCB, SW22 SW_Cherry_MX_1.00u_PCB, SW23 SW_Cherry_MX_1.00u_PCB, SW24 SW_Cherry_MX_1.00u_PCB, SW25 SW_Cherry_MX_1.00u_PCB, SW26 SW_Cherry_MX_1.50u_PCB, SW27 SW_Cherry_MX_1.00u_PCB, SW28 SW_Cherry_MX_1.00u_PCB, SW29 SW_Cherry_MX_1.00u_PCB, SW3 SW_Cherry_MX_1.00u_PCB, SW30 SW_Cherry_MX_1.00u_PCB, SW31 SW_Cherry_MX_1.00u_PCB, SW32 SW_Cherry_MX_1.00u_PCB, SW33 SW_Cherry_MX_1.00u_PCB, SW34 SW_Cherry_MX_1.00u_PCB, SW35 SW_Cherry_MX_1.00u_PCB, SW36 SW_Cherry_MX_1.00u_PCB, SW37 SW_Cherry_MX_1.00u_PCB, SW38 SW_Cherry_MX_1.00u_PCB, SW39 SW_Cherry_MX_1.00u_PCB, SW4 SW_Cherry_MX_1.00u_PCB, SW40 SW_Cherry_MX_1.00u_PCB, SW41 SW_Cherry_MX_1.50u_PCB, SW42 SW_Cherry_MX_1.00u_PCB, SW43 SW_Cherry_MX_1.00u_PCB, SW44 SW_Cherry_MX_1.00u_PCB, SW45 SW_Cherry_MX_1.00u_PCB, SW46 SW_Cherry_MX_1.00u_PCB, SW47 SW_Cherry_MX_1.00u_PCB, SW48 SW_Cherry_MX_1.00u_PCB, SW49 SW_Cherry_MX_1.00u_PCB, SW5 SW_Cherry_MX_1.00u_PCB, SW50 SW_Cherry_MX_1.00u_PCB, SW51 SW_Cherry_MX_1.00u_PCB, SW52 SW_Cherry_MX_1.50u_PCB, SW53 SW_Cherry_MX_1.00u_PCB, SW6 SW_Cherry_MX_1.00u_PCB, SW7 SW_Cherry_MX_1.00u_PCB, SW8 SW_Cherry_MX_1.00u_PCB, SW9 SW_Cherry_MX_1.00u_PCB, U10 27C16 / 2816, U11 27C16 / 2816, U12 27C16 / 2816, U13 27C16 / 2816, U14 6850, U15 74LS02, U16 74LS04, U17 74LS159, U18 74LS04, U19 74LS20, U2 74LS75, U20 74LS138, U21 74LS04, U22 74LS138, U23 74LS138, U24 8T28, U25 8T28, U29 74LS93, U3 74LS75, U30 74LS163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

Commit message: checking for shorts
Connections:
- U36 pad 18: (no net) -> Vcc
- U36 pad 9: (no net) -> GND
- U37 pad 18: (no net) -> Vcc
- U37 pad 9: (no net) -> GND
Routing:
- net (no net): track 50588.3 -> 40249.7 mm, vias 647 -> 521
- net Vcc: track 111.8 -> 10450.4 mm, vias 6 -> 132
